Commit message: Revise Rover Model

File: model/mcl_rover/assets/urdf/Rover_3D_YCM.urdf (robot description, URDF)
Before this commit: robot Rover_3D_YCM, 17 links, 16 joints
Links:
- link FL_bot_sus_bar: mass 0.187287611019615 -> 5.56431340636313
- link FL_steer_link: mass 0.0918924650288386 -> 2.73012416238969
- link FL_sus_cover: mass 0.0574115008234622 -> 1.70569522443191
- link FL_wheel: mass 6.43655550433335 -> 5.00003734648168
- link FR_bot_sus_bar: mass 0.187287611019615 -> 5.56431340636313
- link FR_steer_link: mass 0.0918924614280398 -> 2.73012416238976
- link FR_sus_cover: mass 0.0574115008234622 -> 1.70569522443191
- link FR_wheel: mass 6.43655550433335 -> 5.00003734648169
- link RL_bot_sus_bar: mass 0.187287611019616 -> 5.56431340636312
- link RL_steer_link: mass 0.0918924614280402 -> 2.73012416238971
- link RL_sus_cover: mass 0.0574115008234622 -> 1.70569522443191
- link RL_wheel: mass 6.43655550433335 -> 5.00003734648169
- link RR_bot_sus_bar: mass 0.187287611019616 -> 5.56431340636313
- link RR_steer_link: mass 0.0918924650288373 -> 2.73012416238972
- link RR_sus_cover: mass 0.0574115008234622 -> 1.70569522443191
- link RR_wheel: mass 6.43655550433335 -> 5.00003734648168
- link base_link: mass 1.33511107631683 -> 94
Joints:
- joint FL_drive_act: origin xyz=-0.08 0 -0.05 rpy=3.1416 -1.5708 0 -> xyz=-0.0799999999999998 0 -0.0500000000000003 rpy=3.14159265358979 -1.5707963267949 0
- joint FL_steer_rev: origin xyz=-0.029978 0.0011562 0 rpy=1.5708 0 0 -> xyz=-0.03 0 0 rpy=1.5707963267949 0 0
- joint FL_sus_act: origin xyz=0.58735 -0.88 -0.042158 rpy=-1.5708 0 -1.5708 -> xyz=0.54 0.21 0.0400000000000001 rpy=-1.5707963267949 0 -1.5707963267949
- joint FL_sus_link_joint: origin xyz=-0.1599 -0.0055723 0.005 rpy=0 0 0 -> xyz=-0.16 0 0.00500000000000023 rpy=0 0 0
- joint FR_drive_act: origin xyz=0.08 0 -0.05 rpy=-1.5508 0.84128 1.5857 -> xyz=0.0800000000000005 0 -0.0499999999999821 rpy=-1.5707963267949 0 1.5707963267949
- joint FR_steer_rev: origin xyz=0.03 0 0 rpy=1.5708 0 0 -> xyz=0.0299999999999996 0 0 rpy=1.5707963267949 0 0
- joint FR_sus_act: origin xyz=0.58735 -1.3 -0.042158 rpy=-1.5708 0 -1.5708 -> xyz=0.54 -0.21 0.04 rpy=-1.5707963267949 0 -1.5707963267949
- joint FR_sus_link_joint: origin xyz=0.15999 -0.0021361 0.005 rpy=0 0 0 -> xyz=0.160000000000002 0 0.005 rpy=0 0 0
- joint RL_drive_act: origin xyz=-0.08 0 -0.05 rpy=3.1416 -1.5708 0 -> xyz=-0.0800000000000001 0 -0.05 rpy=3.14159265358979 -1.5707963267949 0
- joint RL_steer_rev: origin xyz=-0.03 0 0 rpy=1.5708 0 0 -> xyz=-0.03 0 0 rpy=1.5707963267949 0 0
- joint RL_sus_act: origin xyz=-0.49265 -0.88 -0.042158 rpy=-1.5708 0 -1.5708 -> xyz=-0.54 0.21 0.04 rpy=-1.5707963267949 0 -1.5707963267949
- joint RL_sus_link_joint: origin xyz=-0.15986 -0.0066568 -0.005 rpy=0 0 0 -> xyz=-0.16 0 -0.00500000000000012 rpy=0 0 0
- joint RR_steer_rev: axis 0 0 1 -> 0 0 -1; origin xyz=0.03 0 0 rpy=1.5706 0 0 -> xyz=0.0300000000000002 0 0 rpy=1.5707963267949 0 0
- joint RR_sus_act: origin xyz=-0.49265 -1.3 -0.042158 rpy=-1.5708 0 -1.5708 -> xyz=-0.54 -0.21 0.04 rpy=-1.5707963267949 0 -1.5707963267949
- joint RR_sus_link_joint: origin xyz=0.16 -0.0006196 -0.005 rpy=0 0 0 -> xyz=0.16 0 -0.00500000000000012 rpy=0 0 0
- joint Rr_drive_act: origin xyz=0.080193 0 -0.04969 rpy=1.5747 0 -1.5708 -> xyz=0.0800000000000001 0 -0.0500000000000001 rpy=1.5707963267949 0 -1.5707963267949
